File: BoardFiles/TopBoard/photonNixieTop.brd (EAGLE design)
At the start: 100 x 35.2 mm, 16 parts, among them J1 2X6 FEMALE

Commit message: Code and case changes
Parts:
- turned D1 to 180 degrees
- turned D2 to 180 degrees
- turned D3 to 180 degrees
- turned D4 to 180 degrees
Connections:
- net GND renamed 5V
- net BLUELED: now also D1.A, D2.A, D3.A, D4.A; no longer D1.C, D2.C, D3.C, D4.C
- net N$2: now also D4.C, R4.2; no longer D1.A, R1.2
- net N$3: now also D3.C, R3.2; no longer D2.A, R2.2
- net N$4: now also D2.C, R2.2; no longer D3.A, R3.2
- net N$5: now also D1.C, R1.2; no longer D4.A, R4.2
Routing:
- net 5V: track 143.9 -> 150.9 mm
- net N$2: track 3.60 -> 1.67 mm
